File: BMW-IABS-Converter.kicad_pcb (KiCad board)
At the start: 2 copper layers, 41 parts, among them J1 SWD, Q1 IRLML0060TRPbF, Q2 IRLML0060TRPbF, Q3 IRFR9024, Q4 IRFR9024, U1 LM358, U2 LM358, U3 LM358, U4 LM358

Commit message: Updated schematics
Parts:
- removed the Q4 at (152.8, 100.2)
- removed R11: 10R, Resistor_SMD:R_0402_1005Metric
- removed R12, R15: 10K, Resistor_SMD:R_0402_1005Metric
- removed U4: LM358, Package_SO:SOIC-8_3.9x4.9mm_P1.27mm
- added Q6: IRFR9024, Package_TO_SOT_SMD:TO-252-2, F.Cu at (146.4, 75.1)
- added R13: 200R, Capacitor_SMD:C_0402_1005Metric, F.Cu at (141.8, 80.1)
- C11: value 1uF -> 10uF
- R14: value 10R -> 200R; footprint Resistor_SMD:R_0402_1005Metric -> Capacitor_SMD:C_0402_1005Metric
- R17: renamed from R13; value 1K -> 100R
- U1: value LM358 -> SN65HVD230
- U2: value LM358 -> STM32F042F4P6
- U3: value LM358 -> MC34063AD
- moved R14 36.7 mm to (153.9, 76.6)
- moved D6 30.0 mm to (156.5, 73.4)
- renumbered Q3 to Q4
Connections:
- C11 pad 1: Net-(C11-Pad1) -> /TAS
- C11 pad 2: (no net) -> /SPEED_PWM
- Q4 pad 2: +12V -> /58RL
- Q4 pad 3: /58RL -> +12V
- R17 pad 1: Net-(C11-Pad1) -> /TAS
- U2 pad 13: (no net) -> /SPEED_PWM
- U2 pad 8: (no net) -> /SPEED_PWM

Commit message: Added connector footprint and symbol
Parts:
- added C9: 330uF (EZV331M0JRC8), Capacitor_SMD:CP_Elec_6.3x7.7, F.Cu at (148.3, 115.7)
- added J2: HCCPHPE24BKA90F, HCCPHPE24BKA90F:HCCPHPE24BKA90F, F.Cu at (191.0, 97.5)
- added NT1: 15 Tie, NetTie:NetTie-2_SMD_Pad0.5mm, F.Cu at (147.5, 80.2)
- added NT2: TA- Tie, NetTie:NetTie-2_SMD_Pad0.5mm, F.Cu at (150.5, 80.2)
- added R11: 1K, Resistor_SMD:R_0603_1608Metric, F.Cu at (148.0, 77.9)
- added R12: 1K, Resistor_SMD:R_0603_1608Metric, F.Cu at (152.0, 77.9)
- added U4: LM2904, Package_SO:SOIC-8_3.9x4.9mm_P1.27mm, F.Cu at (157.7, 114.9)
- C11: value 10uF -> 1uF
- R17: value 100R -> 1K
- moved D1 22.6 mm to (118.2, 104.5)
- moved J1 22.6 mm to (124.4, 87.1)
- moved C1 22.6 mm to (129.0, 94.4)
- moved C10 22.6 mm to (129.3, 109.2)
- moved C11 22.6 mm to (154.8, 102.1)
- moved C2 22.6 mm to (144.1, 88.9)
- moved C3 22.6 mm to (132.5, 114.3)
- moved C5 22.6 mm to (126.8, 114.3)
- moved C6 22.6 mm to (144.6, 110.4)
- moved C7 22.6 mm to (153.7, 104.3)
- moved C8 22.6 mm to (136.6, 111.7)
- moved D2 22.6 mm to (148.7, 95.2)
- moved D3 22.6 mm to (148.7, 99.8)
- moved D4 22.6 mm to (138.6, 108.1)
- moved D6 22.6 mm to (133.9, 74.2)
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Connections:
- D3 pad 1: +12V -> /15U
- Q2 pad 3: (no net) -> /ABS-W
- R13 pad 2: (no net) -> Net-(R13-Pad2)
- R14 pad 2: (no net) -> Net-(R14-Pad2)
- R8 pad 2: (no net) -> /GEN_WARN
- U2 pad 10: (no net) -> /TAIL_LIGHT
- U2 pad 11: (no net) -> /GEN_WARN
- U2 pad 9: (no net) -> /BRAKE_LIGHT
